File: carte lidar.kicad_sch (KiCad schematic)
At the start: 15 parts, among them J1 UART CP, J2 LIDAR, J3 XBEE, J8 alim, U1 XIAO-ESP32-S3-DIP

Commit message: condo et qq changement
Parts:
- C1: footprint Capacitor_THT:CP_Radial_D10.0mm_P5.00mm -> Capacitor_THT:CP_Radial_D5.0mm_P2.00mm
Changed lines of the file:
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@@
 			)
 		)
-		(property "Footprint" "Capacitor_THT:CP_Radial_D10.0mm_P5.00mm"
+		(property "Footprint" "Capacitor_THT:CP_Radial_D5.0mm_P2.00mm"
 			(at 130.81 34.29 0)
 			(effects
