File: carte lidar.kicad_pcb (KiCad board)
At the start: 2 copper layers, 40 x 40 mm, 15 parts, among them J1 UART CP, J2 LIDAR, J3 XBEE, J8 alim, U1 XIAO-ESP32-S3-DIP

Commit message: fix
Parts:
- D1, J3: moved to B.Cu
- moved J3 10.7 mm to (136.2, 65.0)
- moved J2 5.50 mm to (145.0, 60.0)
Routing:
- net +3.3V: track 22.9 -> 40.7 mm
- net TX XBEE: track 12.0 -> 25.9 mm
- net RX XBEE: track 12.8 -> 23.6 mm
- net +5V: track 51.7 -> 56.5 mm
- net Lidar_PWM: track 15.1 -> 19.1 mm
- net RX LIDAR: track 8.94 -> 6.57 mm
- net TX LIDAR: track 8.82 -> 6.53 mm
- added copper zone on B.Cu, net GND

Commit message: etiquettes
Parts:
- added kibuzzard-67ED5E55: G***, kibuzzard-67ED5E55, B.Cu at (146.0, 39.5)
- added kibuzzard-67ED5E55: G***, kibuzzard-67ED5E55, B.Cu at (141.4, 42.4)
- added kibuzzard-67ED8412: G***, kibuzzard-67ED8412, B.Cu at (146.3, 52.2)
- added kibuzzard-67ED8456: G***, kibuzzard-67ED8456, B.Cu at (146.0, 49.7)
- added kibuzzard-68F1EF6D: G***, kibuzzard-68F1EF6D, F.Cu at (140.1, 54.5)
- added kibuzzard-68F1EFC1: G***, kibuzzard-68F1EFC1, F.Cu at (127.8, 37.5)
- added kibuzzard-68F1EFDA: G***, kibuzzard-68F1EFDA, B.Cu at (145.8, 65.0)
- added kibuzzard-68F1EFE5: G***, kibuzzard-68F1EFE5, F.Cu at (148.1, 59.8)
- added kibuzzard-68F1F041: G***, kibuzzard-68F1F041, F.Cu at (157.1, 43.5)
- added kibuzzard-68F1F0CD: G***, kibuzzard-68F1F0CD, F.Cu at (152.4, 36.9)
- added kibuzzard-68F1F1A3: G***, kibuzzard-68F1F1A3, B.Cu at (146.0, 37.0)
- added kibuzzard-68F1F1EA: G***, kibuzzard-68F1F1EA, B.Cu at (135.9, 37.0)
- added kibuzzard-68F1F1F6: G***, kibuzzard-68F1F1F6, B.Cu at (135.9, 39.5)
- added kibuzzard-68F1F236: G***, kibuzzard-68F1F236, B.Cu at (135.6, 42.1)
- added kibuzzard-68F1F243: G***, kibuzzard-68F1F243, B.Cu at (135.6, 44.6)
- added kibuzzard-68F1F26D: G***, kibuzzard-68F1F26D, B.Cu at (145.4, 42.1)
- added kibuzzard-68F1F2E0: G***, kibuzzard-68F1F2E0, B.Cu at (133.9, 52.2)
- added kibuzzard-68F1F3B3: G***, kibuzzard-68F1F3B3, B.Cu at (155.0, 42.4)

Commit message: v2 un poil violent XD
Parts:
- removed kibuzzard-67ED5E55 (x2): G***, kibuzzard-67ED5E55
- removed kibuzzard-67ED8412: G***, kibuzzard-67ED8412
- removed kibuzzard-67ED8456: G***, kibuzzard-67ED8456
- removed kibuzzard-68F1EF6D: G***, kibuzzard-68F1EF6D
- removed kibuzzard-68F1EFC1: G***, kibuzzard-68F1EFC1
- removed kibuzzard-68F1EFDA: G***, kibuzzard-68F1EFDA
- removed kibuzzard-68F1EFE5: G***, kibuzzard-68F1EFE5
- removed kibuzzard-68F1F041: G***, kibuzzard-68F1F041
- removed kibuzzard-68F1F0CD: G***, kibuzzard-68F1F0CD
- removed kibuzzard-68F1F1A3: G***, kibuzzard-68F1F1A3
- removed kibuzzard-68F1F1EA: G***, kibuzzard-68F1F1EA
- removed kibuzzard-68F1F1F6: G***, kibuzzard-68F1F1F6
- removed kibuzzard-68F1F236: G***, kibuzzard-68F1F236
- removed kibuzzard-68F1F243: G***, kibuzzard-68F1F243
- removed kibuzzard-68F1F26D: G***, kibuzzard-68F1F26D
- removed kibuzzard-68F1F2E0: G***, kibuzzard-68F1F2E0
- removed kibuzzard-68F1F3B3: G***, kibuzzard-68F1F3B3
- D1, J3, R4, R5: moved to F.Cu
- D2, R2: moved to B.Cu
- moved R2 48.5 mm to (107.0, 55.2)
- moved J8 46.1 mm to (108.3, 50.5), turned to 180 degrees
- moved D2 45.0 mm to (107.0, 57.8), turned to 180 degrees
- moved J2 40.1 mm to (106.7, 72.0), turned to 90 degrees
- moved J1 38.9 mm to (100.2, 72.3)
- moved H3 37.5 mm to (126.0, 72.0)
- moved J3 37.1 mm to (100.2, 55.7), turned to -90 degrees
- moved R1 36.4 mm to (112.5, 71.0), turned to 0 degrees
- moved R3 33.1 mm to (112.5, 68.5), turned to 0 degrees
- moved R4 32.1 mm to (107.0, 55.2), turned to 0 degrees
- moved R5 29.9 mm to (107.0, 57.8), turned to 0 degrees
- moved D1 25.8 mm to (124.8, 48.8)
- moved U1 24.2 mm to (119.8, 57.8)
- moved H2 24.0 mm to (100.0, 50.2)
- moved C1 21.8 mm to (122.1, 56.2), turned to 180 degrees
Connections:
- R4 pad 1: TX XBEE -> RX XBEE
- R5 pad 1: RX XBEE -> TX XBEE
Routing:
- net Lidar_PWM: track 19.1 -> 39.8 mm, vias 0 -> 1
- net TX XBEE: track 25.9 -> 6.41 mm
- net RX XBEE: track 23.6 -> 5.39 mm
- net +3.3V: track 40.7 -> 50.7 mm
- net UART CPS: track 12.5 -> 22.4 mm
- net Net-(U1-GPIO3/D2/A2): track 13.0 -> 3.60 mm
- net Net-(D2-A): track 8.62 -> 2.56 mm
- net Net-(U1-GPIO4/D3/A3): track 8.89 -> 3.58 mm
- net +5V: track 56.5 -> 51.8 mm
- net UART CPE: track 29.4 -> 32.3 mm
- net GND: track 2.77 -> 0.00 mm
- net RX LIDAR: track 6.57 -> 4.85 mm
- net TX LIDAR: track 6.53 -> 4.85 mm
- net Net-(U1-GPIO1/D0/A0): track 21.0 -> 22.7 mm
- net Net-(D1-K): track 4.39 -> 3.11 mm
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- added copper zone on F.Cu, net GND
Other:
- board size 40 x 40 mm -> 34 x 30 mm

Commit message: begining logo
Parts:
- added G***: LOGO, LOGO, B.Cu at (119.9, 58.9)
- added kibuzzard-690B60FE: G***, kibuzzard-690B60FE, F.Cu at (113.7, 52.7)
- added kibuzzard-690B60FE: G***, kibuzzard-690B60FE, F.Cu at (113.8, 65.4)
- added kibuzzard-690B60FE: G***, kibuzzard-690B60FE, F.Cu at (113.7, 57.7)
- added kibuzzard-690B6108: G***, kibuzzard-690B6108, F.Cu at (125.7, 65.4)
- added kibuzzard-690B6148: G***, kibuzzard-690B6148, F.Cu at (123.5, 62.8)
- added kibuzzard-690B618A: G***, kibuzzard-690B618A, F.Cu at (113.7, 50.2)
- added kibuzzard-690B618A: G***, kibuzzard-690B618A, F.Cu at (113.7, 55.2)
- moved C1 0.47 mm to (122.3, 56.7)
Routing:
- net +5V: track 51.8 -> 51.1 mm
Other:
- board text added: "By Oscar Yosh GRIVELET"
- board text added: "Carte_lidar 2026_V2"

Commit message: fix
Routing:
- net UART CPE: track 32.3 -> 31.5 mm
Changed lines of the file:
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@@
 			(psa4output no)
 			(plot_black_and_white yes)
-			(plotinvisibletext no)
 			(sketchpadsonfab no)
 			(plotpadnumbers no)
@@
 				(font
 					(size 0.001 0.001)
+					(thickness 0.15)
 				)
 			)
@@
 				(font
 					(size 0.001 0.001)
+					(thickness 0.15)
 				)
 			)
@@
 				(font
 					(size 0.001 0.001)
+					(thickness 0.15)
 				)
 			)
@@
 				(font
 					(size 0.001 0.001)
+					(thickness 0.15)
 				)
 			)
@@
 				(font
 					(size 0.001 0.001)
+					(thickness 0.15)
 				)
 			)
@@
 				(font
 					(size 0.001 0.001)
+					(thickness 0.15)
 				)
 			)
@@
 				(font
 					(size 0.001 0.001)
+					(thickness 0.15)
 				)
 			)
@@
 				(font
 					(size 0.001 0.001)
+					(thickness 0.15)
 				)
 			)
@@
 		)
 	)
+	(dimension
+		(type orthogonal)
+		(layer "Dwgs.User")
+		(pts
+			(xy 104.5 46.25) (xy 105.025 76.25)
+		)
+		(height -16.75)
+		(orientation 1)
+		(format
+			(prefix "")
+			(suffix "")
+			(units 3)
+			(units_format 0)
+			(precision 4)
+			(suppress_zeroes yes)
+		)
+		(style
+			(thickness 0.15)
+			(arrow_length 1.27)
+			(text_position_mode 0)
+			(arrow_direction outward)
+			(extension_height 0.58642)
+			(extension_offset 0.5)
+			(keep_text_aligned yes)
+		)
+		(gr_text "30"
+			(at 86.6 61.25 90)
+			(layer "Dwgs.User")
+			(effects
+				(font
+					(size 1 1)
+					(thickness 0.15)
+				)
+			)
+		)
+	)
+	(dimension
+		(type orthogonal)
+		(layer "Dwgs.User")
+		(pts
+			(xy 96 64.71) (xy 130 64.887776)
+		)
+		(height -25.21)
+		(orientation 0)
+		(format
+			(prefix "")
+			(suffix "")
+			(units 3)
+			(units_format 0)
+			(precision 4)
+			(suppress_zeroes yes)
+		)
+		(style
+			(thickness 0.15)
+			(arrow_length 1.27)
+			(text_position_mode 0)
+			(arrow_direction outward)
+			(extension_height 0.58642)
+			(extension_offset 0.5)
+			(keep_text_aligned yes)
+		)
+		(gr_text "34"
+			(at 113 38.35 0)
+			(layer "Dwgs.User")
+			(effects
+				(font
+					(size 1 1)
+					(thickness 0.15)
+				)
+			)
+		)
+	)
 	(segment
 		(start 122.117677 65.632323)
@@
 	)
 	(segment
-		(start 122.625 67.125)
-		(end 115.85 73.9)
+		(start 106 62)
+		(end 106.725 62)
 		(width 0.5)
 		(layer "F.Cu")
@@
 	)
 	(segment
-		(start 106 73.9)
-		(end 105 72.9)
+		(start 122.625 67.125)
+		(end 116.3 73.45)
 		(width 0.5)
 		(layer "F.Cu")
@@
 	)
 	(segment
-		(start 105 63)
-		(end 106 62)
+		(start 105.55 73.45)
+		(end 105 72.9)
 		(width 0.5)
 		(layer "F.Cu")
@@
 	)
 	(segment
-		(start 122.75 66.875)
-		(end 122.625 67)
+		(start 105 63)
+		(end 106 62)
 		(width 0.5)
 		(layer "F.Cu")
@@
 	)
 	(segment
-		(start 115.85 73.9)
-		(end 106 73.9)
+		(start 116.3 73.45)
+		(end 105.55 73.45)
 		(width 0.5)
 		(layer "F.Cu")
@@
 	)
 	(segment
-		(start 106 62)
-		(end 106.725 62)
+		(start 122.625 67)
+		(end 122.625 67.125)
 		(width 0.5)
 		(layer "F.Cu")
@@
 	)
 	(segment
-		(start 122.625 67)
-		(end 122.625 67.125)
+		(start 122.75 66.875)
+		(end 122.625 67)
 		(width 0.5)
 		(layer "F.Cu")
@@
 	)
 	(segment
-		(start 124 67.5)
-		(end 116.7 74.8)
+		(start 101.08 63.33)
+		(end 100.25 63.33)
 		(width 0.5)
 		(layer "F.Cu")
@@
 	)
 	(segment
-		(start 127.37 55.21)
-		(end 128.205 55.21)
+		(start 124 58.58)
+		(end 124 67.5)
 		(width 0.5)
 		(layer "F.Cu")
@@
 	)
 	(segment
-		(start 104 66.25)
-		(end 101.08 63.33)
+		(start 124 67.5)
+		(end 117.3 74.2)
 		(width 0.5)
 		(layer "F.Cu")
@@
 	)
 	(segment
-		(start 101.08 63.33)
-		(end 100.25 63.33)
+		(start 127.37 55.21)
+		(end 128.205 55.21)
 		(width 0.5)
 		(layer "F.Cu")
@@
 	)
 	(segment
-		(start 127.37 55.21)
-		(end 124 58.58)
+		(start 117.3 74.2)
+		(end 104.7 74.2)
 		(width 0.5)
 		(layer "F.Cu")
@@
 	)
 	(segment
-		(start 124 58.58)
-		(end 124 67.5)
+		(start 104.7 74.2)
+		(end 104 73.5)
 		(width 0.5)
 		(layer "F.Cu")
@@
 	)
 	(segment
-		(start 105.3 74.8)
-		(end 104 73.5)
+		(start 104 66.25)
+		(end 101.08 63.33)
 		(width 0.5)
 		(layer "F.Cu")
@@
 	)
 	(segment
-		(start 104 73.5)
-		(end 104 66.25)
+		(start 127.37 55.21)
+		(end 124 58.58)
 		(width 0.5)
 		(layer "F.Cu")
@@
 	)
 	(segment
-		(start 116.7 74.8)
-		(end 105.3 74.8)
+		(start 104 73.5)
+		(end 104 66.25)
 		(width 0.5)
 		(layer "F.Cu")
@@
 	)
 	(segment
-		(start 127.37 65.37)
-		(end 127.13 65.37)
+		(start 101.91 74.2)
+		(end 100.25 72.54)
 		(width 0.5)
 		(layer "B.Cu")
@@
 	)
 	(segment
-		(start 117.25 75.25)
-		(end 102.96 75.25)
+		(start 127.37 65.37)
+		(end 127.13 65.37)
 		(width 0.5)
 		(layer "B.Cu")
@@
 	)
 	(segment
-		(start 102.96 75.25)
-		(end 100.25 72.54)
+		(start 127.13 65.37)
+		(end 118.3 74.2)
 		(width 0.5)
 		(layer "B.Cu")
@@
 	)
 	(segment
-		(start 127.13 65.37)
-		(end 117.25 75.25)
+		(start 118.3 74.2)
+		(end 101.91 74.2)
 		(width 0.5)
 		(layer "B.Cu")
@@
 	)
 	(segment
-		(start 112.5 65.74)
-		(end 112.5 72.75)
+		(start 112.5 72.75)
+		(end 111.8 73.45)
 		(width 0.5)
 		(layer "B.Cu")
@@
 	)
 	(segment
-		(start 112.13 65.37)
-		(end 112.5 65.74)
+		(start 112.5 65.74)
+		(end 112.5 72.75)
 		(width 0.5)
 		(layer "B.Cu")
@@
 	)
 	(segment
-		(start 112.5 72.75)
-		(end 111.25 74)
+		(start 112.13 65.37)
+		(end 112.5 65.74)
 		(width 0.5)
 		(layer "B.Cu")
@@
 	)
 	(segment
-		(start 100.75 70)
-		(end 100.25 70)
+		(start 111.8 73.45)
+		(end 104.2 73.45)
 		(width 0.5)
 		(layer "B.Cu")
@@
 	)
 	(segment
-		(start 104.75 74)
+		(start 104.2 73.45)
 		(end 100.75 70)
 		(width 0.5)
@@
 	)
 	(segment
-		(start 111.25 74)
-		(end 104.75 74)
+		(start 100.75 70)
+		(end 100.25 70)
 		(width 0.5)
 		(layer "B.Cu")
@@
 		(polygon
 			(pts
-				(xy 130 46.25) (xy 95.998795 46.181821) (xy 95.998795 76.251205) (xy 130 76.251205)
+				(xy 130 46.25) (xy 95.95 46.181821) (xy 95.998795 76.251205) (xy 130 76.251205)
 			)
 		)

Commit message: condo et qq changement
Parts:
- C1: footprint Capacitor_THT:CP_Radial_D10.0mm_P5.00mm -> Capacitor_THT:CP_Radial_D5.0mm_P2.00mm
- moved C1 3.10 mm to (122.4, 53.6), turned to 0 degrees
- moved G*** 1.16 mm to (119.8, 57.8)
Routing:
- net GND: track 0.00 -> 153.7 mm
- net +5V: track 51.1 -> 53.6 mm

Commit message: ayaaaa
Parts:
- moved C1 6.40 mm to (116.0, 53.6)
Routing:
- net +5V: track 53.6 -> 42.6 mm
- net GND: track 153.7 -> 147.4 mm
Changed lines of the file:
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@@
 			(psa4output no)
 			(plot_black_and_white yes)
-			(plotinvisibletext no)
 			(sketchpadsonfab no)
 			(plotpadnumbers no)
@@
 			(pinfunction "Pin_3")
 			(pintype "passive")
+			(thermal_bridge_angle 45)
 		)
 		(embedded_fonts no)
@@
 	(footprint "Capacitor_THT:CP_Radial_D5.0mm_P2.00mm"
 		(layer "F.Cu")
-		(at 122.399999 53.6)
+		(at 115.999999 53.6)
 		(descr "CP, Radial series, Radial, pin pitch=2.00mm, , diameter=5mm, Electrolytic Capacitor")
 		(tags "CP Radial series Radial pin pitch 2.00mm  diameter 5mm Electrolytic Capacitor")
@@
 			(pinfunction "Pin_3")
 			(pintype "passive")
+			(thermal_bridge_angle 45)
 		)
 		(pad "4" thru_hole oval
@@
 			(pinfunction "Pin_4")
 			(pintype "passive")
+			(thermal_bridge_angle 45)
 		)
 		(pad "5" thru_hole oval
@@
 			(pinfunction "Pin_2")
 			(pintype "passive")
+			(thermal_bridge_angle 45)
 		)
 		(embedded_fonts no)
@@
 	)
 	(segment
-		(start 125.33 52.67)
-		(end 124.4 53.6)
-		(width 0.8)
-		(layer "B.Cu")
-		(net 1)
-	)
-	(segment
 		(start 108.7 64.5)
 		(end 106.725 64.5)
@@
 	)
 	(segment
-		(start 124.4 52.46863)
-		(end 124.4 53.6)
-		(width 0.8)
-		(layer "B.Cu")
-		(net 1)
-	)
-	(segment
 		(start 102.96 64.5)
 		(end 100.25 67.21)
@@
 	)
 	(segment
-		(start 123.140685 51.209315)
-		(end 124.4 52.46863)
-		(width 0.8)
-		(layer "B.Cu")
-		(net 1)
-	)
-	(segment
 		(start 118.88237 46.951)
 		(end 123.140685 51.209315)
@@
 	)
 	(segment
-		(start 127.37 52.67)
-		(end 125.33 52.67)
-		(width 0.8)
-		(layer "B.Cu")
-		(net 1)
-	)
-	(segment
 		(start 97.6 67.1)
 		(end 97.6 73.35)
@@
 	)
 	(segment
-		(start 122.399999 51.799999)
-		(end 122.399999 64.800001)
-		(width 0.8)
-		(layer "F.Cu")
-		(net 2)
-	)
-	(segment
-		(start 114.67 48.75)
-		(end 119.35 48.75)
+		(start 110.2 72)
+		(end 106.725 72)
 		(width 0.8)
 		(layer "F.Cu")
@@
 	)
 	(segment
-		(start 115.2 72)
-		(end 106.725 72)
+		(start 115.999999 50.079999)
+		(end 115.999999 66.200001)
 		(width 0.8)
 		(layer "F.Cu")
@@
 	)
 	(segment
-		(start 122.399999 64.800001)
-		(end 115.2 72)
-		(width 0.8)
-		(layer "F.Cu")
-		(net 2)
-	)
-	(segment
 		(start 108.275 50.48)
 		(end 108.275 49.475)
@@
 	)
 	(segment
+		(start 114.67 48.75)
+		(end 115.999999 50.079999)
+		(width 0.8)
+		(layer "F.Cu")
+		(net 2)
+	)
+	(segment
 		(start 109 48.5)
 		(end 114.42 48.5)
@@
 	)
 	(segment
-		(start 119.35 48.75)
-		(end 122.399999 51.799999)
+		(start 115.999999 66.200001)
+		(end 110.2 72)
 		(width 0.8)
 		(layer "F.Cu")

Commit message: silkscreen
Parts:
- added kibuzzard-690E9271: G***, kibuzzard-690E9271, F.Cu at (107.0, 47.1)
- added kibuzzard-690E93B3: G***, kibuzzard-690E93B3, B.Cu at (107.0, 57.0)
- added kibuzzard-690E9406: G***, kibuzzard-690E9406, F.Cu at (107.0, 57.2)
- added kibuzzard-690E9406: G***, kibuzzard-690E9406, F.Cu at (107.0, 54.7)
- added kibuzzard-690E9406: G***, kibuzzard-690E9406, B.Cu at (112.5, 68.0)
- added kibuzzard-690E9406: G***, kibuzzard-690E9406, B.Cu at (107.0, 54.7)
- added kibuzzard-690E9406: G***, kibuzzard-690E9406, B.Cu at (112.5, 70.5)
- added kibuzzard-690E943A: G***, kibuzzard-690E943A, F.Cu at (107.0, 55.8)
- added kibuzzard-690E943A: G***, kibuzzard-690E943A, F.Cu at (107.0, 58.2)
- added kibuzzard-690E943A: G***, kibuzzard-690E943A, B.Cu at (112.5, 71.5)
- added kibuzzard-690E943A: G***, kibuzzard-690E943A, B.Cu at (112.5, 69.0)
- added kibuzzard-690E943A: G***, kibuzzard-690E943A, B.Cu at (107.0, 55.8)
- added kibuzzard-6915AC9B: G***, kibuzzard-6915AC9B, F.Cu at (96.9, 59.5)
- added kibuzzard-6915ACBE: G***, kibuzzard-6915ACBE, F.Cu at (96.8, 69.8)
- added kibuzzard-6915AD2C: G***, kibuzzard-6915AD2C, B.Cu at (104.6, 67.0)
- added kibuzzard-6915AD46: G***, kibuzzard-6915AD46, B.Cu at (104.6, 69.5)
- added kibuzzard-6915AD82: G***, kibuzzard-6915AD82, B.Cu at (98.0, 55.7)
- added kibuzzard-6915AD88: G***, kibuzzard-6915AD88, B.Cu at (98.0, 58.2)
- added kibuzzard-6915ADA8: G***, kibuzzard-6915ADA8, B.Cu at (98.0, 72.3)
- added kibuzzard-6915ADB1: G***, kibuzzard-6915ADB1, B.Cu at (98.0, 69.8)
- added kibuzzard-6915ADC6: G***, kibuzzard-6915ADC6, F.Cu at (106.7, 75.0)
- moved H3 0.25 mm to (126.0, 72.2)
